File: hardware/small_oscilloscope/audio.kicad_sch (KiCad schematic)
At the start: 6 parts, among them J4 Conn_01x02, U4 LM358

Commit message: 250627 circuit
Parts:
- C10: renamed from C6; value 20n -> 20p; footprint (none) -> Capacitor_SMD:C_0402_1005Metric_Pad0.74x0.62mm_HandSolder
- J6: renamed from J4; footprint Connector_PinSocket_2.54mm:PinSocket_1x02_P2.54mm_Vertical -> Connector_PinHeader_2.54mm:PinHeader_1x04_P2.54mm_Vertical
- R44: renamed from R23; footprint (none) -> Resistor_SMD:R_0603_1608Metric_Pad0.98x0.95mm_HandSolder
- R45: renamed from R26; footprint (none) -> Resistor_SMD:R_0402_1005Metric_Pad0.72x0.64mm_HandSolder
- R46: renamed from R27; footprint (none) -> Resistor_SMD:R_0402_1005Metric_Pad0.72x0.64mm_HandSolder
- U12: renamed from U4; footprint (none) -> Package_DIP:DIP-8_W7.62mm_LongPads
Changed lines of the file:
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@@
 		(dnp no)
 		(fields_autoplaced yes)
-		(property "Reference" "J4"
+		(property "Reference" "J6"
 			(at 172.72 87.6299 0)
 			(effects
@@
 			)
 		)
-		(property "Footprint" "Connector_PinSocket_2.54mm:PinSocket_1x02_P2.54mm_Vertical"
+		(property "Footprint" "Connector_PinHeader_2.54mm:PinHeader_1x04_P2.54mm_Vertical"
 			(at 170.18 87.63 0)
 			(effects
@@
 		)
 		(instances
-			(project ""
-				(path "/722ad30e-a672-4959-92bf-662e54054c44/361d5bc8-a591-4e5d-9bf7-7ac2147493e8"
-					(reference "J4")
+			(project "small_oscilloscope"
+				(path "/722ad30e-a672-4959-92bf-662e54054c44/cef6da11-c0f0-4933-af38-0fa8b3242acf/40985c4a-08eb-4c1d-83fc-6aefc7584ddd"
+					(reference "J6")
 					(unit 1)
 				)
@@
 		(dnp no)
 		(fields_autoplaced yes)
-		(property "Reference" "R26"
+		(property "Reference" "R45"
 			(at 114.3 93.9799 0)
 			(effects
@@
 			)
 		)
-		(property "Footprint" ""
+		(property "Footprint" "Resistor_SMD:R_0402_1005Metric_Pad0.72x0.64mm_HandSolder"
 			(at 109.982 95.25 90)
 			(effects
@@
 		)
 		(instances
-			(project ""
-				(path "/722ad30e-a672-4959-92bf-662e54054c44/361d5bc8-a591-4e5d-9bf7-7ac2147493e8"
-					(reference "R26")
+			(project "small_oscilloscope"
+				(path "/722ad30e-a672-4959-92bf-662e54054c44/cef6da11-c0f0-4933-af38-0fa8b3242acf/40985c4a-08eb-4c1d-83fc-6aefc7584ddd"
+					(reference "R45")
 					(unit 1)
 				)
@@
 		(dnp no)
 		(fields_autoplaced yes)
-		(property "Reference" "R27"
+		(property "Reference" "R46"
 			(at 114.3 107.9499 0)
 			(effects
@@
 			)
 		)
-		(property "Footprint" ""
+		(property "Footprint" "Resistor_SMD:R_0402_1005Metric_Pad0.72x0.64mm_HandSolder"
 			(at 109.982 109.22 90)
 			(effects
@@
 		(instances
 			(project "small_oscilloscope"
-				(path "/722ad30e-a672-4959-92bf-662e54054c44/361d5bc8-a591-4e5d-9bf7-7ac2147493e8"
-					(reference "R27")
+				(path "/722ad30e-a672-4959-92bf-662e54054c44/cef6da11-c0f0-4933-af38-0fa8b3242acf/40985c4a-08eb-4c1d-83fc-6aefc7584ddd"
+					(reference "R46")
 					(unit 1)
 				)
@@
 		(dnp no)
 		(fields_autoplaced yes)
-		(property "Reference" "R23"
+		(property "Reference" "R44"
 			(at 66.04 59.69 90)
 			(effects
@@
 			)
 		)
-		(property "Footprint" ""
+		(property "Footprint" "Resistor_SMD:R_0603_1608Metric_Pad0.98x0.95mm_HandSolder"
 			(at 66.04 67.818 90)
 			(effects
@@
 		)
 		(instances
-			(project ""
-				(path "/722ad30e-a672-4959-92bf-662e54054c44/361d5bc8-a591-4e5d-9bf7-7ac2147493e8"
-					(reference "R23")
+			(project "small_oscilloscope"
+				(path "/722ad30e-a672-4959-92bf-662e54054c44/cef6da11-c0f0-4933-af38-0fa8b3242acf/40985c4a-08eb-4c1d-83fc-6aefc7584ddd"
+					(reference "R44")
 					(unit 1)
 				)
@@
 		(dnp no)
 		(fields_autoplaced yes)
-		(property "Reference" "#PWR046"
+		(property "Reference" "#PWR094"
 			(at 93.98 121.92 0)
 			(effects
@@
 		)
 		(instances
-			(project ""
-				(path "/722ad30e-a672-4959-92bf-662e54054c44/361d5bc8-a591-4e5d-9bf7-7ac2147493e8"
-					(reference "#PWR046")
+			(project "small_oscilloscope"
+				(path "/722ad30e-a672-4959-92bf-662e54054c44/cef6da11-c0f0-4933-af38-0fa8b3242acf/40985c4a-08eb-4c1d-83fc-6aefc7584ddd"
+					(reference "#PWR094")
 					(unit 1)
 				)
@@
 		(dnp no)
 		(fields_autoplaced yes)
-		(property "Reference" "U4"
+		(property "Reference" "U12"
 			(at 95.25 101.5999 0)
 			(effects
@@
 			)
 		)
-		(property "Footprint" ""
+		(property "Footprint" "Package_DIP:DIP-8_W7.62mm_LongPads"
 			(at 96.52 102.87 0)
 			(effects
@@
 		)
 		(instances
-			(project ""
-				(path "/722ad30e-a672-4959-92bf-662e54054c44/361d5bc8-a591-4e5d-9bf7-7ac2147493e8"
-					(reference "U4")
+			(project "small_oscilloscope"
+				(path "/722ad30e-a672-4959-92bf-662e54054c44/cef6da11-c0f0-4933-af38-0fa8b3242acf/40985c4a-08eb-4c1d-83fc-6aefc7584ddd"
+					(reference "U12")
 					(unit 3)
 				)
@@
 		(dnp no)
 		(fields_autoplaced yes)
-		(property "Reference" "U4"
+		(property "Reference" "U12"
 			(at 139.7 58.42 0)
 			(effects
@@
 			)
 		)
-		(property "Footprint" ""
+		(property "Footprint" "Package_DIP:DIP-8_W7.62mm_LongPads"
 			(at 139.7 68.58 0)
 			(effects
@@
 		(instances
 			(project "small_oscilloscope"
-				(path "/722ad30e-a672-4959-92bf-662e54054c44/361d5bc8-a591-4e5d-9bf7-7ac2147493e8"
-					(reference "U4")
+				(path "/722ad30e-a672-4959-92bf-662e54054c44/cef6da11-c0f0-4933-af38-0fa8b3242acf/40985c4a-08eb-4c1d-83fc-6aefc7584ddd"
+					(reference "U12")
 					(unit 1)
 				)
@@
 		(dnp no)
 		(fields_autoplaced yes)
-		(property "Reference" "#PWR047"
+		(property "Reference" "#PWR093"
 			(at 73.66 90.17 0)
 			(effects
@@
 		(instances
 			(project "small_oscilloscope"
-				(path "/722ad30e-a672-4959-92bf-662e54054c44/361d5bc8-a591-4e5d-9bf7-7ac2147493e8"
-					(reference "#PWR047")
+				(path "/722ad30e-a672-4959-92bf-662e54054c44/cef6da11-c0f0-4933-af38-0fa8b3242acf/40985c4a-08eb-4c1d-83fc-6aefc7584ddd"
+					(reference "#PWR093")
 					(unit 1)
 				)
@@
 		(dnp no)
 		(fields_autoplaced yes)
-		(property "Reference" "#PWR048"
+		(property "Reference" "#PWR095"
 			(at 111.76 125.73 0)
 			(effects
@@
 		(instances
 			(project "small_oscilloscope"
-				(path "/722ad30e-a672-4959-92bf-662e54054c44/361d5bc8-a591-4e5d-9bf7-7ac2147493e8"
-					(reference "#PWR048")
+				(path "/722ad30e-a672-4959-92bf-662e54054c44/cef6da11-c0f0-4933-af38-0fa8b3242acf/40985c4a-08eb-4c1d-83fc-6aefc7584ddd"
+					(reference "#PWR095")
 					(unit 1)
 				)
@@
 		(dnp no)
 		(fields_autoplaced yes)
-		(property "Reference" "U4"
+		(property "Reference" "U12"
 			(at 139.7 93.98 0)
 			(effects
@@
 			)
 		)
-		(property "Footprint" ""
+		(property "Footprint" "Package_DIP:DIP-8_W7.62mm_LongPads"
 			(at 139.7 104.14 0)
 			(effects
@@
 		)
 		(instances
-			(project ""
-				(path "/722ad30e-a672-4959-92bf-662e54054c44/361d5bc8-a591-4e5d-9bf7-7ac2147493e8"
-					(reference "U4")
+			(project "small_oscilloscope"
+				(path "/722ad30e-a672-4959-92bf-662e54054c44/cef6da11-c0f0-4933-af38-0fa8b3242acf/40985c4a-08eb-4c1d-83fc-6aefc7584ddd"
+					(reference "U12")
 					(unit 2)
 				)
@@
 		(dnp no)
 		(fields_autoplaced yes)
-		(property "Reference" "C6"
+		(property "Reference" "C10"
 			(at 77.47 72.3899 0)
 			(effects
@@
 			)
 		)
-		(property "Value" "20n"
+		(property "Value" "20p"
 			(at 77.47 74.9299 0)
 			(effects
@@
 			)
 		)
-		(property "Footprint" ""
+		(property "Footprint" "Capacitor_SMD:C_0402_1005Metric_Pad0.74x0.62mm_HandSolder"
 			(at 74.6252 77.47 0)
 			(effects
@@
 		)
 		(instances
-			(project ""
-				(path "/722ad30e-a672-4959-92bf-662e54054c44/361d5bc8-a591-4e5d-9bf7-7ac2147493e8"
-					(reference "C6")
-					(unit 1)
-				)
+			(project "small_oscilloscope"
+				(path "/722ad30e-a672-4959-92bf-662e54054c44/cef6da11-c0f0-4933-af38-0fa8b3242acf/40985c4a-08eb-4c1d-83fc-6aefc7584ddd"
+					(reference "C10")
+					(unit 1)
+				)

Commit message: feat: 오실로스코프 회로 설계 업데이트
Parts:
- J6: footprint Connector_PinHeader_2.54mm:PinHeader_1x04_P2.54mm_Vertical -> Connector_PinHeader_2.54mm:PinHeader_1x02_P2.54mm_Vertical
Changed lines of the file:
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@@
 			)
 		)
-		(property "Footprint" "Connector_PinHeader_2.54mm:PinHeader_1x04_P2.54mm_Vertical"
+		(property "Footprint" "Connector_PinHeader_2.54mm:PinHeader_1x02_P2.54mm_Vertical"
 			(at 170.18 87.63 0)
 			(effects

Commit message: oscilliscope first success
Parts:
- C14: renamed from C10; now left out of the parts list
- J6: value Conn_01x02 -> SPEAKER; footprint Connector_PinHeader_2.54mm:PinHeader_1x02_P2.54mm_Vertical -> Connector_PinSocket_2.54mm:PinSocket_1x02_P2.54mm_Vertical; now left out of the parts list
- R90: renamed from R44; now left out of the parts list
- R91: renamed from R45; now left out of the parts list
- R92: renamed from R46; now left out of the parts list
- U13: renamed from U12; footprint Package_DIP:DIP-8_W7.62mm_LongPads -> Package_SO:SOIC-8_3.9x4.9mm_P1.27mm; now left out of the parts list
Changed lines of the file:
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@@
 		(unit 1)
 		(exclude_from_sim no)
-		(in_bom yes)
+		(in_bom no)
 		(on_board yes)
 		(dnp no)
@@
 			)
 		)
-		(property "Value" "Conn_01x02"
+		(property "Value" "SPEAKER"
 			(at 172.72 90.1699 0)
 			(effects
@@
 			)
 		)
-		(property "Footprint" "Connector_PinHeader_2.54mm:PinHeader_1x02_P2.54mm_Vertical"
+		(property "Footprint" "Connector_PinSocket_2.54mm:PinSocket_1x02_P2.54mm_Vertical"
 			(at 170.18 87.63 0)
 			(effects
@@
 		(unit 1)
 		(exclude_from_sim no)
-		(in_bom yes)
-		(on_board yes)
-		(dnp no)
-		(fields_autoplaced yes)
-		(property "Reference" "R45"
+		(in_bom no)
+		(on_board yes)
+		(dnp no)
+		(fields_autoplaced yes)
+		(property "Reference" "R91"
 			(at 114.3 93.9799 0)
 			(effects
@@
 			(project "small_oscilloscope"
 				(path "/722ad30e-a672-4959-92bf-662e54054c44/cef6da11-c0f0-4933-af38-0fa8b3242acf/40985c4a-08eb-4c1d-83fc-6aefc7584ddd"
-					(reference "R45")
+					(reference "R91")
 					(unit 1)
 				)
@@
 		(unit 1)
 		(exclude_from_sim no)
-		(in_bom yes)
-		(on_board yes)
-		(dnp no)
-		(fields_autoplaced yes)
-		(property "Reference" "R46"
+		(in_bom no)
+		(on_board yes)
+		(dnp no)
+		(fields_autoplaced yes)
+		(property "Reference" "R92"
 			(at 114.3 107.9499 0)
 			(effects
@@
 			(project "small_oscilloscope"
 				(path "/722ad30e-a672-4959-92bf-662e54054c44/cef6da11-c0f0-4933-af38-0fa8b3242acf/40985c4a-08eb-4c1d-83fc-6aefc7584ddd"
-					(reference "R46")
+					(reference "R92")
 					(unit 1)
 				)
@@
 		(unit 1)
 		(exclude_from_sim no)
-		(in_bom yes)
-		(on_board yes)
-		(dnp no)
-		(fields_autoplaced yes)
-		(property "Reference" "R44"
+		(in_bom no)
+		(on_board yes)
+		(dnp no)
+		(fields_autoplaced yes)
+		(property "Reference" "R90"
 			(at 66.04 59.69 90)
 			(effects
@@
 			(project "small_oscilloscope"
 				(path "/722ad30e-a672-4959-92bf-662e54054c44/cef6da11-c0f0-4933-af38-0fa8b3242acf/40985c4a-08eb-4c1d-83fc-6aefc7584ddd"
-					(reference "R44")
+					(reference "R90")
 					(unit 1)
 				)
@@
 		(dnp no)
 		(fields_autoplaced yes)
-		(property "Reference" "#PWR094"
+		(property "Reference" "#PWR0146"
 			(at 93.98 121.92 0)
 			(effects
@@
 			(project "small_oscilloscope"
 				(path "/722ad30e-a672-4959-92bf-662e54054c44/cef6da11-c0f0-4933-af38-0fa8b3242acf/40985c4a-08eb-4c1d-83fc-6aefc7584ddd"
-					(reference "#PWR094")
+					(reference "#PWR0146")
 					(unit 1)
 				)
@@
 		(unit 3)
 		(exclude_from_sim no)
-		(in_bom yes)
-		(on_board yes)
-		(dnp no)
-		(fields_autoplaced yes)
-		(property "Reference" "U12"
+		(in_bom no)
+		(on_board yes)
+		(dnp no)
+		(fields_autoplaced yes)
+		(property "Reference" "U13"
 			(at 95.25 101.5999 0)
 			(effects
@@
 			)
 		)
-		(property "Footprint" "Package_DIP:DIP-8_W7.62mm_LongPads"
+		(property "Footprint" "Package_SO:SOIC-8_3.9x4.9mm_P1.27mm"
 			(at 96.52 102.87 0)
 			(effects
@@
 			(project "small_oscilloscope"
 				(path "/722ad30e-a672-4959-92bf-662e54054c44/cef6da11-c0f0-4933-af38-0fa8b3242acf/40985c4a-08eb-4c1d-83fc-6aefc7584ddd"
-					(reference "U12")
+					(reference "U13")
 					(unit 3)
 				)
@@
 		(unit 1)
 		(exclude_from_sim no)
-		(in_bom yes)
-		(on_board yes)
-		(dnp no)
-		(fields_autoplaced yes)
-		(property "Reference" "U12"
+		(in_bom no)
+		(on_board yes)
+		(dnp no)
+		(fields_autoplaced yes)
+		(property "Reference" "U13"
 			(at 139.7 58.42 0)
 			(effects
@@
 			)
 		)
-		(property "Footprint" "Package_DIP:DIP-8_W7.62mm_LongPads"
+		(property "Footprint" "Package_SO:SOIC-8_3.9x4.9mm_P1.27mm"
 			(at 139.7 68.58 0)
 			(effects
@@
 			(project "small_oscilloscope"
 				(path "/722ad30e-a672-4959-92bf-662e54054c44/cef6da11-c0f0-4933-af38-0fa8b3242acf/40985c4a-08eb-4c1d-83fc-6aefc7584ddd"
-					(reference "U12")
+					(reference "U13")
 					(unit 1)
 				)
@@
 		(dnp no)
 		(fields_autoplaced yes)
-		(property "Reference" "#PWR093"
+		(property "Reference" "#PWR0145"
 			(at 73.66 90.17 0)
 			(effects
@@
 			(project "small_oscilloscope"
 				(path "/722ad30e-a672-4959-92bf-662e54054c44/cef6da11-c0f0-4933-af38-0fa8b3242acf/40985c4a-08eb-4c1d-83fc-6aefc7584ddd"
-					(reference "#PWR093")
+					(reference "#PWR0145")
 					(unit 1)
 				)
@@
 		(dnp no)
 		(fields_autoplaced yes)
-		(property "Reference" "#PWR095"
+		(property "Reference" "#PWR0147"
 			(at 111.76 125.73 0)
 			(effects
@@
 			(project "small_oscilloscope"
 				(path "/722ad30e-a672-4959-92bf-662e54054c44/cef6da11-c0f0-4933-af38-0fa8b3242acf/40985c4a-08eb-4c1d-83fc-6aefc7584ddd"
-					(reference "#PWR095")
+					(reference "#PWR0147")
 					(unit 1)
 				)
@@
 		(unit 2)
 		(exclude_from_sim no)
-		(in_bom yes)
-		(on_board yes)
-		(dnp no)
-		(fields_autoplaced yes)
-		(property "Reference" "U12"
+		(in_bom no)
+		(on_board yes)
+		(dnp no)
+		(fields_autoplaced yes)
+		(property "Reference" "U13"
 			(at 139.7 93.98 0)
 			(effects
@@
 			)
 		)
-		(property "Footprint" "Package_DIP:DIP-8_W7.62mm_LongPads"
+		(property "Footprint" "Package_SO:SOIC-8_3.9x4.9mm_P1.27mm"
 			(at 139.7 104.14 0)
 			(effects
@@
 			(project "small_oscilloscope"
 				(path "/722ad30e-a672-4959-92bf-662e54054c44/cef6da11-c0f0-4933-af38-0fa8b3242acf/40985c4a-08eb-4c1d-83fc-6aefc7584ddd"
-					(reference "U12")
+					(reference "U13")
 					(unit 2)
 				)
@@
 		(unit 1)
 		(exclude_from_sim no)
-		(in_bom yes)
-		(on_board yes)
-		(dnp no)
-		(fields_autoplaced yes)
-		(property "Reference" "C10"
+		(in_bom no)
+		(on_board yes)
+		(dnp no)
+		(fields_autoplaced yes)
+		(property "Reference" "C14"
 			(at 77.47 72.3899 0)
 			(effects
@@
 			(project "small_oscilloscope"
 				(path "/722ad30e-a672-4959-92bf-662e54054c44/cef6da11-c0f0-4933-af38-0fa8b3242acf/40985c4a-08eb-4c1d-83fc-6aefc7584ddd"
-					(reference "C10")
-					(unit 1)
-				)
+					(reference "C14")
+					(unit 1)
+				)
