File: hardware/small_oscilloscope/lcd.kicad_sch (KiCad schematic)
At the start: 7 parts, among them J5 Parellel LCD, Q9 NTR5103NT1G, U11 FT800Q-T, Y1 12.0000M

Commit message: feat: 오실로스코프 회로 설계 업데이트
Parts:
- J5: footprint Connector_PinHeader_2.54mm:PinHeader_1x04_P2.54mm_Vertical -> Connector_FFC-FPC:TE_4-1734839-0_1x40-1MP_P0.5mm_Horizontal
- R43: value 1K -> 1k; footprint Resistor_THT:R_Axial_DIN0207_L6.3mm_D2.5mm_P10.16mm_Horizontal -> Resistor_SMD:R_0603_1608Metric_Pad0.98x0.95mm_HandSolder
Connections:
- net +24V: now also J5.39 (LEDA); no longer J5.2 (LEDA)
- net +3.3V: now also J5.37 (VDD); no longer J5.4 (VDD)
- net GND: now also J5.12 (GND), J5.38 (GND), J5.5 (GND), J5.6 (NC), J5.MP, U11.49 (EPAD); no longer J5.29 (GND), J5.3 (GND), J5.35 (NC), J5.36 (GND), U11.EPAD
- net at U11.19 (X+): now also J5.4 (XR); no longer J5.37 (XR)
- net at U11.20 (Y+): now also J5.3 (YD); no longer J5.38 (YD)
- net at U11.21 (X-): now also J5.2 (XL); no longer J5.39 (XL)
- net at U11.22 (Y-): now also J5.1 (YU); no longer J5.40 (YU)
- net at U11.25 (DE): now also J5.7 (DE); no longer J5.34 (DE)
- net at U11.26 (VSYNC): now also J5.8 (VSYNC); no longer J5.33 (VSYNC)
- net at U11.27 (HSYNC): now also J5.9 (HSYNC); no longer J5.32 (HSYNC)
- net at U11.28 (DISP): now also J5.10 (DISP); no longer J5.31 (DISP)
- net at U11.29 (PCLK): now also J5.11 (DCLK); no longer J5.30 (DCLK)
- net at U11.30 (B7): now also J5.13 (B7); no longer J5.28 (B7)
- net at U11.31 (B6): now also J5.14 (B6); no longer J5.27 (B6)
- net at U11.32 (B5): now also J5.15 (B5); no longer J5.26 (B5)
- net at U11.33 (B4): now also J5.16 (B4); no longer J5.25 (B4)
- net at U11.34 (B3): now also J5.17 (B3); no longer J5.24 (B3)
- net at J5.20 (B0): now also J5.18 (B2), J5.19 (B1), U11.35 (B2); no longer U11.37 (G7)
- net at U11.38 (G6): now also J5.22 (G6); no longer J5.19 (G6)
- net at U11.39 (G5): now also J5.23 (G5); no longer J5.18 (G5)
- net at U11.40 (G4): now also J5.24 (G4); no longer J5.17 (G4)
- net at U11.41 (G3): now also J5.25 (G3); no longer J5.16 (G3)
- net at U11.43 (R7): now also J5.29 (R7); no longer J5.12 (R7)
- net at U11.44 (R6): now also J5.30 (R6); no longer J5.11 (R6)
- net at U11.45 (R5): now also J5.31 (R5); no longer J5.10 (R5)
- net at U11.46 (R4): now also J5.32 (R4); no longer J5.9 (R4)
- net at U11.47 (R3): now also J5.33 (R3); no longer J5.8 (R3)
- net at Q9.3 (D): now also J5.40 (LEDK); no longer J5.1 (LEDK)
- new net: J5.21 (G7), U11.37 (G7)
- new net: J5.26 (G2), J5.27 (G1), J5.28 (G0), U11.42 (G2)
- new net: J5.34 (R2), J5.35 (R1), J5.36 (R0), U11.48 (R2)
Changed lines of the file:
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@@
+	)
+	(junction
+		(at 203.2 134.62)
+		(diameter 0)
+		(color 0 0 0 0)
 	)
 	(junction
@@
 	(wire
 		(pts
+			(xy 203.2 134.62) (xy 203.2 121.92)
+		)
+		(stroke
+			(width 0)
+			(type default)
+		)
+	)
+	(wire
+		(pts
 			(xy 185.42 43.18) (xy 205.74 43.18)
 		)
@@
 	(wire
 		(pts
+			(xy 203.2 134.62) (xy 205.74 134.62)
+		)
+		(stroke
+			(width 0)
+			(type default)
+		)
+	)
+	(wire
+		(pts
 			(xy 185.42 48.26) (xy 205.74 48.26)
 		)
@@
 	(wire
 		(pts
-			(xy 203.2 137.16) (xy 203.2 121.92)
+			(xy 203.2 137.16) (xy 203.2 134.62)
 		)
 		(stroke
@@
 			)
 		)
-		(property "Value" "1K"
+		(property "Value" "1k"
 			(at 58.42 80.0099 0)
 			(effects
@@
 			)
 		)
-		(property "Footprint" "Resistor_THT:R_Axial_DIN0207_L6.3mm_D2.5mm_P10.16mm_Horizontal"
+		(property "Footprint" "Resistor_SMD:R_0603_1608Metric_Pad0.98x0.95mm_HandSolder"
 			(at 54.102 78.74 90)
 			(effects
@@
 		(pin "23"
 		)
-		(pin "EPAD"
+		(pin "49"
 		)
 		(pin "20"
@@
 			)
 		)
-		(property "Footprint" "Connector_PinHeader_2.54mm:PinHeader_1x04_P2.54mm_Vertical"
+		(property "Footprint" "Connector_FFC-FPC:TE_4-1734839-0_1x40-1MP_P0.5mm_Horizontal"
 			(at 209.55 145.542 0)
 			(effects
@@
 		(pin "40"
 		)
+		(pin "MP"
+		)
 		(instances

Commit message: board edit
Parts:
- U11: footprint Package_DFN_QFN:VQFN-48-1EP_6x6mm_P0.4mm_EP4.1x4.1mm_ThermalVias -> Package_DFN_QFN:VQFN-48-1EP_7x7mm_P0.5mm_EP4.1x4.1mm
Changed lines of the file:
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@@
 			)
 		)
-		(property "Footprint" "Package_DFN_QFN:VQFN-48-1EP_6x6mm_P0.4mm_EP4.1x4.1mm_ThermalVias"
+		(property "Footprint" "Package_DFN_QFN:VQFN-48-1EP_7x7mm_P0.5mm_EP4.1x4.1mm"
 			(at 127 129.54 0)
 			(effects

Commit message: oscilliscope first success
Parts:
- removed Q9: NTR5103NT1G, Package_TO_SOT_SMD:SOT-23_Handsoldering, symbol Transistor_FET:Q_NMOS_GSD
- added C13: 10u, Capacitor_SMD:CP_Elec_5x5.3, symbol Device:C_Polarized
- added R80: 150, Resistor_SMD:R_0402_1005Metric_Pad0.72x0.64mm_HandSolder, symbol Device:R
- added R81, R82: 10k, Resistor_SMD:R_0402_1005Metric_Pad0.72x0.64mm_HandSolder, symbol Device:R
- added R83, R84, R85, R86, R87: 10R, Resistor_SMD:R_1206_3216Metric_Pad1.30x1.75mm_HandSolder, symbol Device:R
- C11: renamed from C8; now left out of the parts list
- C12: renamed from C9; now left out of the parts list
- J5, Y1: now left out of the parts list
- R89: renamed from R43; value 1k -> 10k; footprint Resistor_SMD:R_0603_1608Metric_Pad0.98x0.95mm_HandSolder -> Resistor_SMD:R_0402_1005Metric_Pad0.72x0.64mm_HandSolder; now left out of the parts list
- U12: renamed from U11; now left out of the parts list
Connections:
- net +24V: now also R80.1; no longer J5.39 (LEDA)
- net +3.3V: now also R81.1, R82.1; no longer U12.17 (VCC1V2)
- net CS: now also R86.1; no longer U12.6 (CS_N/_I2C_SA1)
- net GND: now also J5.40 (LEDK), C13.2; no longer J5.6 (NC)
- net MISO: now also R84.1; no longer U12.4 (MISO/_I2C_SDA)
- net MOSI: now also R85.1; no longer U12.5 (MOSI/_I2C_SA0)
- net SCLK: now also R83.1; no longer U12.3 (SPI_SCLK/_I2C_SCL)
- net at U12.11 (INT_N): now also R81.2, R87.2
- net at U12.12 (PD_N): now also R82.2
- new net: R86.2, U12.6 (CS_N/_I2C_SA1)
- new net: R83.2, U12.3 (SPI_SCLK/_I2C_SCL)
- new net: C13.1, U12.17 (VCC1V2)
- new net: R84.2, U12.4 (MISO/_I2C_SDA)
- new net: R85.2, U12.5 (MOSI/_I2C_SA0)
- new net: J5.39 (LEDA), R80.2
- new net ~{INT}: R87.1
Other:
- moved on the sheet: R89
